Commit message: modified

File: war_ws/src/war_description/urdf/conveyor.xacro (robot description, xacro)
@@ -63,5 +63,5 @@
         </inertial>
     </link>
-    <joint name="front_conveyor_roller_joint" type="continuous">
+    <joint name="front_conveyor_roller_joint" type="fixed">
         <parent link="conveyor_frame"/>
         <child link="front_conveyor_roller"/>
@@ -90,5 +90,5 @@
         </inertial>
     </link>
-    <joint name="rear_conveyor_roller_joint" type="continuous">
+    <joint name="rear_conveyor_roller_joint" type="fixed">
         <parent link="conveyor_frame"/>
         <child link="rear_conveyor_roller"/>
